File: kicad/nRFControlPanel/nRFControlPanel.kicad_sch (KiCad schematic)
At the start: 11 parts, among them J1 Power, J2 Digital/PWM, J3 Analog, J4 Digital/PWM, SW1 SW_Push, SW2 SW_Push, SW4 SW_Push, U1 RC1602A, U2 NRF24L01_Breakout

Commit message: more work on the schematic for the nRFControlPanel
Connections:
- net +5V: now also U1.2 (VDD)
- net GND: now also R1.2
Other:
- moved on the sheet: U2
Changed lines of the file:
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@@
     (date "mar. 31 mars 2015")
   )
-  (junction (at 123.19 24.13) (diameter 0) (color 0 0 0 0)
-  )
   (junction (at 31.75 46.99) (diameter 1.016) (color 0 0 0 0)
   )
   (junction (at 97.79 92.71) (diameter 0) (color 0 0 0 0)
   )
-  (junction (at 109.22 24.13) (diameter 0) (color 0 0 0 0)
-  )
   (junction (at 97.79 73.66) (diameter 0) (color 0 0 0 0)
-  )
-  (junction (at 109.22 59.69) (diameter 0) (color 0 0 0 0)
-  )
-  (junction (at 121.92 46.99) (diameter 0) (color 0 0 0 0)
   )
   (no_connect (at 34.29 31.75))
@@
     (stroke (width 0) (type solid))
   )
-  (wire (pts (xy 133.35 24.13) (xy 123.19 24.13))
-    (stroke (width 0) (type default))
-  )
   (wire (pts (xy 62.23 26.67) (xy 74.93 26.67))
     (stroke (width 0) (type solid))
   )
-  (wire (pts (xy 119.38 49.53) (xy 130.81 49.53))
-    (stroke (width 0) (type default))
-  )
-  (wire (pts (xy 119.38 46.99) (xy 121.92 46.99))
-    (stroke (width 0) (type default))
-  )
   (wire (pts (xy 31.75 44.45) (xy 31.75 46.99))
     (stroke (width 0) (type solid))
@@
     (stroke (width 0) (type solid))
   )
-  (wire (pts (xy 133.35 36.83) (xy 133.35 46.99))
-    (stroke (width 0) (type default))
-  )
   (wire (pts (xy 29.21 41.91) (xy 34.29 41.91))
     (stroke (width 0) (type solid))
@@
     (stroke (width 0) (type solid))
   )
-  (wire (pts (xy 146.05 72.39) (xy 146.05 74.93))
+  (wire (pts (xy 205.74 73.66) (xy 205.74 76.2))
     (stroke (width 0) (type default))
   )
@@
     (stroke (width 0) (type solid))
   )
-  (wire (pts (xy 133.35 31.75) (xy 133.35 24.13))
-    (stroke (width 0) (type default))
-  )
-  (wire (pts (xy 123.19 24.13) (xy 109.22 24.13))
+  (wire (pts (xy 133.35 31.75) (xy 133.35 20.32))
+    (stroke (width 0) (type default))
+  )
+  (wire (pts (xy 133.35 36.83) (xy 133.35 67.31))
     (stroke (width 0) (type default))
   )
@@
     (stroke (width 0) (type solid))
   )
-  (wire (pts (xy 146.05 35.56) (xy 146.05 41.91))
+  (wire (pts (xy 205.74 36.83) (xy 205.74 43.18))
     (stroke (width 0) (type default))
   )
@@
     (stroke (width 0) (type solid))
   )
-  (wire (pts (xy 130.81 46.99) (xy 133.35 46.99))
-    (stroke (width 0) (type default))
-  )
   (wire (pts (xy 21.59 62.23) (xy 34.29 62.23))
     (stroke (width 0) (type solid))
   )
-  (wire (pts (xy 109.22 20.32) (xy 109.22 24.13))
+  (wire (pts (xy 109.22 20.32) (xy 109.22 21.59))
     (stroke (width 0) (type default))
   )
@@
     (stroke (width 0) (type default))
   )
-  (wire (pts (xy 123.19 24.13) (xy 123.19 33.02))
+  (wire (pts (xy 123.19 20.32) (xy 123.19 33.02))
     (stroke (width 0) (type default))
   )
@@
     (stroke (width 0) (type default))
   )
-  (wire (pts (xy 130.81 49.53) (xy 130.81 46.99))
-    (stroke (width 0) (type default))
-  )
   (wire (pts (xy 62.23 64.77) (xy 74.93 64.77))
     (stroke (width 0) (type solid))
   )
-  (wire (pts (xy 123.19 40.64) (xy 123.19 46.99))
-    (stroke (width 0) (type default))
-  )
-  (wire (pts (xy 121.92 46.99) (xy 123.19 46.99))
+  (wire (pts (xy 123.19 40.64) (xy 123.19 67.31))
     (stroke (width 0) (type default))
   )
@@
     (stroke (width 0) (type solid))
   )
-  (wire (pts (xy 121.92 59.69) (xy 109.22 59.69))
-    (stroke (width 0) (type default))
-  )
   (wire (pts (xy 62.23 74.93) (xy 74.93 74.93))
     (stroke (width 0) (type solid))
@@
   )
   (wire (pts (xy 97.79 92.71) (xy 97.79 99.06))
-    (stroke (width 0) (type default))
-  )
-  (wire (pts (xy 121.92 46.99) (xy 121.92 59.69))
     (stroke (width 0) (type default))
   )
@@
     )
   )
-  (symbol (lib_id "power:+3V3") (at 146.05 35.56 0) (unit 1)
-    (in_bom yes) (on_board yes) (dnp no)
-    (property "Reference" "#PWR?" (at 146.05 39.37 0)
-      (effects (font (size 1.27 1.27)) hide)
-    )
-    (property "Value" "+3.3V" (at 146.431 32.512 90)
-      (effects (font (size 1.27 1.27)) (justify left))
-    )
-    (property "Footprint" "" (at 146.05 35.56 0)
-      (effects (font (size 1.27 1.27)))
-    )
-    (property "Datasheet" "" (at 146.05 35.56 0)
+  (symbol (lib_id "power:+5V") (at 123.19 20.32 0) (unit 1)
+    (in_bom yes) (on_board yes) (dnp no)
+    (property "Reference" "#PWR?" (at 123.19 24.13 0)
+      (effects (font (size 1.27 1.27)) hide)
+    )
+    (property "Value" "+5V" (at 123.5456 17.272 90)
+      (effects (font (size 1.27 1.27)) (justify left))
+    )
+    (property "Footprint" "" (at 123.19 20.32 0)
+      (effects (font (size 1.27 1.27)))
+    )
+    (property "Datasheet" "" (at 123.19 20.32 0)
+      (effects (font (size 1.27 1.27)))
+    )
+    (pin "1")
+    (instances
+      (project "nRFControlPanel"
+        (path "/e63e39d7-6ac0-4ffd-8aa3-1841a4541b55"
+          (reference "#PWR?") (unit 1)
+        )
+      )
+    )
+  )
+  (symbol (lib_id "power:+3V3") (at 205.74 36.83 0) (unit 1)
+    (in_bom yes) (on_board yes) (dnp no)
+    (property "Reference" "#PWR?" (at 205.74 40.64 0)
+      (effects (font (size 1.27 1.27)) hide)
+    )
+    (property "Value" "+3.3V" (at 206.121 33.782 90)
+      (effects (font (size 1.27 1.27)) (justify left))
+    )
+    (property "Footprint" "" (at 205.74 36.83 0)
+      (effects (font (size 1.27 1.27)))
+    )
+    (property "Datasheet" "" (at 205.74 36.83 0)
       (effects (font (size 1.27 1.27)))
     )
@@
     )
   )
-  (symbol (lib_id "RF:NRF24L01_Breakout") (at 146.05 57.15 0) (unit 1)
+  (symbol (lib_id "power:+5V") (at 133.35 20.32 0) (unit 1)
+    (in_bom yes) (on_board yes) (dnp no)
+    (property "Reference" "#PWR?" (at 133.35 24.13 0)
+      (effects (font (size 1.27 1.27)) hide)
+    )
+    (property "Value" "+5V" (at 133.7056 17.272 90)
+      (effects (font (size 1.27 1.27)) (justify left))
+    )
+    (property "Footprint" "" (at 133.35 20.32 0)
+      (effects (font (size 1.27 1.27)))
+    )
+    (property "Datasheet" "" (at 133.35 20.32 0)
+      (effects (font (size 1.27 1.27)))
+    )
+    (pin "1")
+    (instances
+      (project "nRFControlPanel"
+        (path "/e63e39d7-6ac0-4ffd-8aa3-1841a4541b55"
+          (reference "#PWR?") (unit 1)
+        )
+      )
+    )
+  )
+  (symbol (lib_id "power:GND") (at 133.35 67.31 0) (unit 1)
+    (in_bom yes) (on_board yes) (dnp no)
+    (property "Reference" "#PWR?" (at 133.35 73.66 0)
+      (effects (font (size 1.27 1.27)) hide)
+    )
+    (property "Value" "GND" (at 133.35 71.12 0)
+      (effects (font (size 1.27 1.27)))
+    )
+    (property "Footprint" "" (at 133.35 67.31 0)
+      (effects (font (size 1.27 1.27)))
+    )
+    (property "Datasheet" "" (at 133.35 67.31 0)
+      (effects (font (size 1.27 1.27)))
+    )
+    (pin "1")
+    (instances
+      (project "nRFControlPanel"
+        (path "/e63e39d7-6ac0-4ffd-8aa3-1841a4541b55"
+          (reference "#PWR?") (unit 1)
+        )
+      )
+    )
+  )
+  (symbol (lib_id "RF:NRF24L01_Breakout") (at 205.74 58.42 0) (unit 1)
     (in_bom yes) (on_board yes) (dnp no) (fields_autoplaced)
-    (property "Reference" "U2" (at 156.21 56.515 0)
-      (effects (font (size 1.27 1.27)) (justify left))
-    )
-    (property "Value" "NRF24L01_Breakout" (at 156.21 59.055 0)
-      (effects (font (size 1.27 1.27)) (justify left))
-    )
-    (property "Footprint" "RF_Module:nRF24L01_Breakout" (at 149.86 41.91 0)
+    (property "Reference" "U2" (at 215.9 57.785 0)
+      (effects (font (size 1.27 1.27)) (justify left))
+    )
+    (property "Value" "NRF24L01_Breakout" (at 215.9 60.325 0)
+      (effects (font (size 1.27 1.27)) (justify left))
+    )
+    (property "Footprint" "RF_Module:nRF24L01_Breakout" (at 209.55 43.18 0)
       (effects (font (size 1.27 1.27) italic) (justify left) hide)
     )
-    (property "Datasheet" "http://www.nordicsemi.com/eng/content/download/2730/34105/file/nRF24L01_Product_Specification_v2_0.pdf" (at 146.05 59.69 0)
+    (property "Datasheet" "http://www.nordicsemi.com/eng/content/download/2730/34105/file/nRF24L01_Product_Specification_v2_0.pdf" (at 205.74 60.96 0)
       (effects (font (size 1.27 1.27)) hide)
     )
@@
     )
   )
-  (symbol (lib_id "power:GND") (at 146.05 74.93 0) (unit 1)
-    (in_bom yes) (on_board yes) (dnp no)
-    (property "Reference" "#PWR?" (at 146.05 81.28 0)
-      (effects (font (size 1.27 1.27)) hide)
-    )
-    (property "Value" "GND" (at 146.05 78.74 0)
-      (effects (font (size 1.27 1.27)))
-    )
-    (property "Footprint" "" (at 146.05 74.93 0)
-      (effects (font (size 1.27 1.27)))
-    )
-    (property "Datasheet" "" (at 146.05 74.93 0)
+  (symbol (lib_id "power:GND") (at 205.74 76.2 0) (unit 1)
+    (in_bom yes) (on_board yes) (dnp no)
+    (property "Reference" "#PWR?" (at 205.74 82.55 0)
+      (effects (font (size 1.27 1.27)) hide)
+    )
+    (property "Value" "GND" (at 205.74 80.01 0)
+      (effects (font (size 1.27 1.27)))
+    )
+    (property "Footprint" "" (at 205.74 76.2 0)
+      (effects (font (size 1.27 1.27)))
+    )
+    (property "Datasheet" "" (at 205.74 76.2 0)
       (effects (font (size 1.27 1.27)))
     )
@@
         )
       )
+    )
+  )
+  (symbol (lib_id "power:GND") (at 123.19 67.31 0) (unit 1)
+    (in_bom yes) (on_board yes) (dnp no)
+    (property "Reference" "#PWR?" (at 123.19 73.66 0)
+      (effects (font (size 1.27 1.27)) hide)
+    )
+    (property "Value" "GND" (at 123.19 71.12 0)
+      (effects (font (size 1.27 1.27)))
+    )
+    (property "Footprint" "" (at 123.19 67.31 0)
+      (effects (font (size 1.27 1.27)))
+    )
+    (property "Datasheet" "" (at 123.19 67.31 0)
+      (effects (font (size 1.27 1.27)))
+    )
+    (pin "1")
+    (instances
+      (project "nRFControlPanel"
+        (path "/e63e39d7-6ac0-4ffd-8aa3-1841a4541b55"
+          (reference "#PWR?") (unit 1)
+        )
+      )
